Commit message: Imported upstream version '0.2.0' of 'upstream'

File: clober_description/urdf/clober.urdf.xacro (robot description, xacro)
@@ -3,10 +3,10 @@
   <!-- <xacro:include filename="$(find clober_description)/urdf/include/tim571.urdf.xacro"/> -->
   <xacro:property name="PI" value="3.1415926535897931"/>
-  <link name="base_footprint"/>
+  <!-- <link name="base_footprint"/>
   <joint name="base_joint" type="fixed">
       <parent link="base_footprint"/>
       <child link="base_link"/>
       <origin xyz="0.0 0.0 0.020" rpy="0 0 0"/>
-  </joint>
+  </joint>     -->
   <link name="base_link">
     <visual>
